Commit message: added collision info in xARM.urdf

File: config/xARM.urdf (robot description, URDF)
Before this commit: robot xARM, 19 links, 18 joints
Links:
- link armlink1_part1: geometry collision box size=0.033 0.003 0.055; visual box size=0.033 0.003 0.055
- link armlink1_part2: geometry collision box size=0.033 0.042 0.003; visual box size=0.033 0.042 0.003
- link armlink1_part3: geometry collision box size=0.033 0.003 0.055; visual box size=0.033 0.003 0.055
- link armlink1_part4: geometry collision cylinder length=0.03 radius=0.0109; visual cylinder length=0.03 radius=0.0109
- link armlink1_part5: geometry collision box size=0.025 0.042 0.003; visual box size=0.025 0.042 0.003
- link armlink1_part6: geometry collision box size=0.025 0.003 0.045; visual box size=0.025 0.003 0.045
- link armlink1_part7: geometry collision box size=0.025 0.003 0.045; visual box size=0.025 0.003 0.045
- link armlink2: geometry collision cylinder length=0.021 radius=0.011435; visual cylinder length=0.021 radius=0.011435
- link armlink3_part1: geometry collision box size=0.04698 0.003 0.06371; visual box size=0.04698 0.003 0.06371
- link armlink3_part2: geometry collision box size=0.04698 0.003 0.06371; visual box size=0.04698 0.003 0.06371
- link armlink4: geometry collision cylinder length=0.022 radius=0.01; visual cylinder length=0.022 radius=0.01
- link base_link: geometry collision box size=0.155 0.14 0.035; visual box size=0.155 0.14 0.035
- link left_gripper: geometry collision box size=0.015 0.015 0.1; visual box size=0.015 0.015 0.1
- link rotary_table: geometry collision cylinder length=0.01 radius=0.06; visual cylinder length=0.01 radius=0.06
- link servo1_link: geometry collision box size=0.05137 0.05682 0.02047; visual box size=0.05137 0.05682 0.02047
- link servo2_link: geometry collision box size=0.04698 0.04250 0.02738; visual box size=0.04698 0.04250 0.02738
- link servo3_link: geometry collision box size=0.02292 0.027 0.04822; visual box size=0.02292 0.027 0.04822
- link servo4_link: geometry collision box size=0.02292 0.027 0.04822; visual box size=0.02292 0.027 0.04822
- link servo5_link: geometry collision box size=0.04402 0.027 0.028; visual box size=0.04402 0.027 0.028

Commit message: Adding counting for the trajectory points received from joint_trajectory_controller

File: config/xARM.urdf (robot description, URDF)
Before this commit: robot xARM, 19 links, 18 joints
Joints:
- joint base_to_rotary_table: limit lower=0.0 upper=4.19 effort=2.0 velocity=0.5 -> lower=-1.5708 upper=1.5708 effort=2.0 velocity=0.5; origin xyz=0 0 0.0175 rpy=0 0 1 -> xyz=0 0 0.035
